Commit message: Removed camera_link

File: desc/franka_description/robots/panda_arm.xacro (robot description, xacro)
@@ -199,5 +199,4 @@
     </joint>
     <link name="${arm_id}_link8"/>
-    <link name="camera_link" />x
     <joint name="${arm_id}_joint8" type="fixed">
       <origin rpy="0 0 0" xyz="0 0 0.107"/>
@@ -205,10 +204,4 @@
       <child link="${arm_id}_link8"/>
       <axis xyz="0 0 0"/>
-    </joint>
-    <joint name="camera_joint" type="fixed">
-      <origin rpy="0 0 0" xyz="0 0 0.0" />
-      <parent link="${arm_id}_link8" />
-      <child link="camera_link" />
-      <axis xyz="0 0 0" />
     </joint>
 <!-- Transmissions of the robot arm - to be able to move each joint ============== -->
