Commit message: Fixed optical frame issue

File: desc/gazebo_description/urdf/depth.xacro (robot description, xacro)
@@ -12,5 +12,5 @@
     </joint>
     <joint name="camera_optical_joint" type="fixed">
-      <origin xyz="0 0 0" rpy="0 0 0" />
+      <origin xyz="0 0 0" rpy="-1.57 0 -1.57" />
       <parent link="camera_link" />
       <child link="${sensor_name}_optical_link" />
