Commit message: Fixed issues, added dimensions and nodes

File: src/projects/table_rearrange/table_rearrange/desc/table_surface.urdf (robot description, URDF)
Before this commit: robot table_surface, 2 links, 1 joints
Links:
- link table: geometry collision box size=0.6 1 0.05; visual box size=0.6 1 0.05

Commit message: Setup grasp pipeline

File: src/projects/table_rearrange/table_rearrange/desc/table_surface.urdf (robot description, URDF)
Before this commit: robot table_surface, 2 links, 1 joints
Links:
- link table: geometry collision box size=0.5 0.5 0.05; visual box size=0.5 0.5 0.05
