Commit message: Fixed end effector location issue

File: src/projects/table_rearrange/table_rearrange/desc/franka_camera.xacro (robot description, xacro)
@@ -8,3 +8,9 @@
 			      parent="panda_link8"
 			      sensor_name="panda_camera"/>
+  <link name="end_effector_link" />
+  <joint name="end_joint" type="fixed">
+    <parent link="panda_hand" />
+    <child link="end_effector_link" />
+    <origin xyz="0 0 0.1" rpy="0 0 0" />
+  </joint>
 </robot>

Commit message: Setup full grasp-place pipeline

File: src/projects/table_rearrange/table_rearrange/desc/franka_camera.xacro (robot description, xacro)
@@ -8,4 +8,5 @@
 			      parent="panda_link8"
 			      sensor_name="panda_camera"/>
+  <!-- Custom additions -->
   <link name="end_effector_link" />
   <joint name="end_joint" type="fixed">
@@ -14,3 +15,17 @@
     <origin xyz="0 0 0.1" rpy="0 0 0" />
   </joint>
+  <gazebo reference="panda_leftfinger">
+    <kp>1000000.0</kp>
+    <kd>1.0</kd>
+    <mu1>1.0</mu1>
+    <mu2>1.0</mu2>
+    <minDepth>0.001</minDepth>
+  </gazebo>
+  <gazebo reference="panda_rightfinger">
+    <kp>1000000.0</kp>
+    <kd>1.0</kd>
+    <mu1>1.0</mu1>
+    <mu2>1.0</mu2>
+    <minDepth>0.001</minDepth>
+  </gazebo>
 </robot>

File: src/projects/table_rearrange/ycb_models/desc/mug.urdf (robot description, URDF)
Before this commit: robot mug, 2 links, 1 joints
Links:
- link mug: mass 1 -> 0.01
