Commit message: Added Lock and Key meshes

File: src/projects/lock_key/lock_key/desc/key.urdf (robot description, URDF)
Before this commit: robot padlock, 2 links, 1 joints
Links:
- removed link padlock
- added link key, mass 0.1; collision mesh filename=package://lock_key/mesh/key.STL; visual mesh filename=package://lock_key/mesh/key.STL
Joints:
- removed joint table_padlock
- added joint table_key: type floating, parent world, child key, origin xyz=0 0 0.05 rpy=0 0 0

Commit message: Added materials and positions

File: src/projects/lock_key/lock_key/desc/key.urdf (robot description, URDF)
Before this commit: robot key, 2 links, 1 joints
Joints:
- joint table_key: origin xyz=0 0 0.05 rpy=0 0 0 -> xyz=-0.32  0.15 0 rpy=1.57 0 1.57

File: src/projects/lock_key/lock_key/desc/padlock.urdf (robot description, URDF)
Before this commit: robot padlock, 2 links, 1 joints
Joints:
- joint table_padlock: origin xyz=0 0 0 rpy=0 0 0 -> xyz=-0.1 0 0 rpy=0 0 1.57
