Commit message: Adding block

File: ros_ws/src/projects/lock_key/lock_key/desc/block.urdf (robot description, URDF)
Before this commit: robot block, 2 links, 1 joints
Joints:
- removed joint table_key
- added joint table_block: type fixed, parent world, child block, origin xyz=-0.105  0.155 0 rpy=0 0 0

File: ros_ws/src/projects/lock_key/lock_key/desc/key.urdf (robot description, URDF)
Before this commit: robot key, 2 links, 1 joints
Joints:
- joint table_key: origin xyz=-0.105  0.155 0.1 rpy=1.57 0 1.57 -> xyz=-0.110  0.165 0.1 rpy=1.57 0 1.57; type fixed -> floating

Commit message: Added Center of Mass

File: ros_ws/src/projects/lock_key/lock_key/desc/block.urdf (robot description, URDF)
Before this commit: robot block, 2 links, 1 joints
Joints:
- joint table_block: origin xyz=-0.105  0.155 0 rpy=0 0 0 -> xyz=0.050000 0.050000 0.050000 rpy=0 0 0; type fixed -> floating

File: ros_ws/src/projects/lock_key/lock_key/desc/key.urdf (robot description, URDF)
Before this commit: robot key, 2 links, 1 joints
Joints:
- joint table_key: origin xyz=-0.110  0.165 0.1 rpy=1.57 0 1.57 -> xyz=0.007250 0.002750 0.030000 rpy=1.57 0 1.57
