Commit message: fixed key issue and segmentation

File: ros_ws/src/projects/lock_key/lock_key/desc/surface.urdf (robot description, URDF)
Before this commit: robot surface, 2 links, 1 joints
Links:
- link table: geometry collision box size=0.6 1 0.005; visual box size=0.6 1 0.001
Joints:
- joint fixed: origin xyz=0.5 0 0.25 rpy=0 0 0 -> xyz=0.75 0 0.25 rpy=0 0 0
