Commit message: Added endeffector link

File: ros_ws/src/projects/lock_key/lock_key/desc/franka_camera.xacro (robot description, xacro)
@@ -5,4 +5,10 @@
   <xacro:include filename="$(find franka_description)/robots/panda_arm_hand.xacro"/>
   <xacro:include filename="$(find gazebo_description)/urdf/depth.xacro" />
+    <link name="end_effector_link" />
+  <joint name="end_joint" type="fixed">
+    <parent link="panda_hand" />
+    <child link="end_effector_link" />
+    <origin xyz="0 0 0.1" rpy="0 0 0" />
+  </joint>
   <xacro:camera_gazebo_sensor xyz="0.05 -0.05 0" rpy="-1.57 -1.57 -0.785"
 			      parent="panda_link8"

Commit message: Added spiral to controller. Added gazebo "attach" plugin
Added gazebo grip stability plugin. Updated spiral trajectory. Added parameters to run.launch. Integrated spiral traj. client with controller.cpp. Created lock_key specific xacros (to include gazebo plugins).

File: ros_ws/src/projects/lock_key/lock_key/desc/franka_camera.xacro (robot description, xacro)
@@ -3,5 +3,5 @@
 <robot xmlns:xacro="http://www.ros.org/wiki/xacro" name="panda_hand_camera">
   <!-- Include xacro files -->
-  <xacro:include filename="$(find franka_description)/robots/panda_arm_hand.xacro"/>
+  <xacro:include filename="$(find franka_description)/robots/panda_arm_hand_lockkey.xacro"/>
   <xacro:include filename="$(find gazebo_description)/urdf/depth.xacro" />
     <link name="end_effector_link" />

File: ros_ws/src/projects/lock_key/lock_key/desc/key.urdf (robot description, URDF)
Before this commit: robot key, 2 links, 1 joints
Joints:
- joint table_key: origin xyz=0.007250 0.002750 0.030000 rpy=1.57 1.57 -1.57 -> xyz=0.007250 0.002750 0.10000 rpy=1.57 1.57 -1.57

File: ros_ws/src/projects/lock_key/lock_key/desc/padlock.urdf (robot description, URDF)
Before this commit: robot padlock, 2 links, 1 joints
Links:
- link padlock: geometry collision mesh filename=package://lock_key/mesh/lock_nominal_002Chamfer.STL; visual mesh filename=package://lock_key/mesh/lock_nominal_002Chamfer.STL
Joints:
- joint table_padlock: origin xyz=-0.1 0 0 rpy=0 0 0 -> xyz=0 0 0 rpy=0 0 0

File: ros_ws/src/projects/lock_key/lock_key/desc/surface.urdf (robot description, URDF)
Before this commit: robot surface, 2 links, 1 joints
Joints:
- joint fixed: origin xyz=0.75 0 0.25 rpy=0 0 0 -> xyz=0.75 0 0.4 rpy=0 0 0
