Commit message: Added block urdf

File: ros_ws/src/projects/lock_key/lock_key/desc/key.urdf (robot description, URDF)
Before this commit: robot key, 2 links, 1 joints
Joints:
- joint table_key: origin xyz=-0.32  0.15 0 rpy=1.57 0 1.57 -> xyz=-0.105  0.155 0.1 rpy=1.57 0 1.57; type floating -> fixed

Commit message: Added key grasping

File: ros_ws/src/projects/lock_key/lock_key/desc/key.urdf (robot description, URDF)
Before this commit: robot key, 2 links, 1 joints
Joints:
- joint table_key: origin xyz=0.007250 0.002750 0.030000 rpy=1.57 0 1.57 -> xyz=0.007250 0.002750 0.030000 rpy=1.57 1.57 1.57

Commit message: lock-key final tuning

File: ros_ws/src/projects/lock_key/lock_key/desc/key.urdf (robot description, URDF)
Before this commit: robot key, 2 links, 1 joints
Links:
- link key: geometry collision box size=0.0145 0.0055 0.06; visual box size=0.0145 0.0055 0.06
Joints:
- joint table_key: origin xyz=0.007250 0.002750 0.030000 rpy=1.57 1.57 1.57 -> xyz=0.007250 0.002750 0.030000 rpy=1.57 1.57 -1.57

File: ros_ws/src/projects/lock_key/lock_key/desc/padlock.urdf (robot description, URDF)
Before this commit: robot padlock, 2 links, 1 joints
Joints:
- joint table_padlock: origin xyz=-0.1 0 0 rpy=0 0 1.57 -> xyz=-0.1 0 0 rpy=0 0 0; type floating -> fixed

Commit message: Fixed collision objects
Fixed collision object definition. Define padlock and key positions as args/params in launch files rather than hardcoding.

File: ros_ws/src/projects/lock_key/lock_key/desc/key.urdf (robot description, URDF)
Before this commit: robot key, 2 links, 1 joints
Joints:
- joint table_key: origin xyz=0.007250 0.002750 0.10000 rpy=1.57 1.57 -1.57 -> xyz=0.0 0.0 0.0 rpy=0.0 0. 0.0
