Commit message: moveit vaguely working

File: ros_ws/src/desc/franka_description/robots/panda_arm_active_vision.xacro (robot description, xacro)
@@ -11,5 +11,5 @@
     <link name="world"/>
     <joint name="fixed" type="fixed">
-      <origin rpy="0 0 0" xyz=".75 0 1"/>
+      <origin rpy="0 0 0" xyz="1.15 0 1.02"/>
       <parent link="world"/>
       <child link="${arm_id}_link0"/>

Commit message: Franka control in simulation success

File: ros_ws/src/desc/franka_description/robots/panda_arm_active_vision.xacro (robot description, xacro)
@@ -11,5 +11,5 @@
     <link name="world"/>
     <joint name="fixed" type="fixed">
-      <origin rpy="0 0 0" xyz="1.15 0 1.02"/>
+      <origin rpy="0 0 0" xyz="1.00 0.00 1.02"/>
       <parent link="world"/>
       <child link="${arm_id}_link0"/>

File: ros_ws/src/projects/active_vision/desc/depth.xacro (robot description, xacro)
@@ -4,5 +4,16 @@
     <!-- joint/link data -->
     <!-- You can modify this to give the camera actual geometry -->
-    <link name="camera_link"></link>
+    <link name="camera_link">>
+      <!-- <inertial>
+       <origin xyz="0 0 0.0" rpy="0 0 0"/>
+       <mass value="0.0001"/>
+       <inertia ixx="0.0001"  ixy="0"  ixz="0" iyy="0.0001" iyz="0" izz="0.0001" />
+     </inertial>
+     <visual>
+       <geometry>
+         <mesh filename="package://active_vision/models/kinectAV/meshes/kinect.dae"/>
+       </geometry>
+     </visual> -->
+    </link>
     <link name="${sensor_name}_optical_link"></link>
     <joint name="robot_camera_joint" type="fixed">
@@ -30,5 +41,5 @@
 	  </image>
 	  <clip>
-	    <near>0.05</near>
+	    <near>0.028</near>
 	    <far>3</far>
 	  </clip>
@@ -46,5 +57,5 @@
           <pointCloudTopicName>/camera/depth/points</pointCloudTopicName>
           <frameName>camera_link</frameName>
-          <pointCloudCutoff>0.5</pointCloudCutoff>
+          <pointCloudCutoff>0.28</pointCloudCutoff>
           <pointCloudCutoffMax>3.0</pointCloudCutoffMax>
           <distortionK1>0</distortionK1>

File: ros_ws/src/projects/active_vision/desc/franka_camera.xacro (robot description, xacro)
@@ -5,5 +5,5 @@
   <xacro:include filename="$(find franka_description)/robots/panda_arm_hand_active_vision.xacro"/>
   <xacro:include filename="$(find active_vision)/desc/depth.xacro" />
-    <link name="end_effector_link" />
+  <link name="end_effector_link" />
   <joint name="end_joint" type="fixed">
     <parent link="panda_hand" />
@@ -11,6 +11,5 @@
     <origin xyz="0 0 0" rpy="0 0 0" />
   </joint>
-  <xacro:camera_gazebo_sensor xyz="0.05 -0.05 0" rpy="-1.57 -1.57 -0.785"
-			      parent="panda_link8"
-			      sensor_name="camera"/>
+  <!-- <xacro:camera_gazebo_sensor xyz="0.05 -0.05 0" rpy="-1.57 -1.57 -0.785" parent="panda_link8" sensor_name="camera"/> -->
+  <xacro:camera_gazebo_sensor xyz="0.06 0 0" rpy="-1.57 -1.57 -1.57" parent="panda_hand" sensor_name="camera"/>
 </robot>

Commit message: Grasp in simulation working

File: ros_ws/src/desc/franka_description/robots/panda_arm_active_vision.xacro (robot description, xacro)
@@ -11,5 +11,5 @@
     <link name="world"/>
     <joint name="fixed" type="fixed">
-      <origin rpy="0 0 0" xyz="1.00 0.00 1.02"/>
+      <origin rpy="0 0 0" xyz="0.00 0.00 0.00"/>
       <parent link="world"/>
       <child link="${arm_id}_link0"/>
@@ -229,9 +229,9 @@
       <type>transmission_interface/SimpleTransmission</type>
       <joint name="${arm_id}_joint1">
-	<hardwareInterface>hardware_interface/EffortJointInterface</hardwareInterface>
+        <hardwareInterface>hardware_interface/EffortJointInterface</hardwareInterface>
       </joint>
       <actuator name="motor1">
-	<hardwareInterface>hardware_interface/EffortJointInterface</hardwareInterface>
-	<mechanicalReduction>1</mechanicalReduction>
+      	<hardwareInterface>hardware_interface/EffortJointInterface</hardwareInterface>
+      	<mechanicalReduction>1</mechanicalReduction>
       </actuator>
     </transmission>
@@ -239,9 +239,9 @@
       <type>transmission_interface/SimpleTransmission</type>
       <joint name="${arm_id}_joint2">
-	<hardwareInterface>hardware_interface/EffortJointInterface</hardwareInterface>
+        <hardwareInterface>hardware_interface/EffortJointInterface</hardwareInterface>
       </joint>
       <actuator name="motor2">
-	<hardwareInterface>hardware_interface/EffortJointInterface</hardwareInterface>
-	<mechanicalReduction>1</mechanicalReduction>
+        <hardwareInterface>hardware_interface/EffortJointInterface</hardwareInterface>
+        <mechanicalReduction>1</mechanicalReduction>
       </actuator>
     </transmission>
@@ -249,9 +249,9 @@
       <type>transmission_interface/SimpleTransmission</type>
       <joint name="${arm_id}_joint3">
-	<hardwareInterface>hardware_interface/EffortJointInterface</hardwareInterface>
+        <hardwareInterface>hardware_interface/EffortJointInterface</hardwareInterface>
       </joint>
       <actuator name="motor3">
-	<hardwareInterface>hardware_interface/EffortJointInterface</hardwareInterface>
-	<mechanicalReduction>1</mechanicalReduction>
+        <hardwareInterface>hardware_interface/EffortJointInterface</hardwareInterface>
+        <mechanicalReduction>1</mechanicalReduction>
       </actuator>
     </transmission>
@@ -259,9 +259,9 @@
       <type>transmission_interface/SimpleTransmission</type>
       <joint name="${arm_id}_joint4">
-	<hardwareInterface>hardware_interface/EffortJointInterface</hardwareInterface>
+        <hardwareInterface>hardware_interface/EffortJointInterface</hardwareInterface>
       </joint>
       <actuator name="motor4">
-	<hardwareInterface>hardware_interface/EffortJointInterface</hardwareInterface>
-	<mechanicalReduction>1</mechanicalReduction>
+        <hardwareInterface>hardware_interface/EffortJointInterface</hardwareInterface>
+        <mechanicalReduction>1</mechanicalReduction>
       </actuator>
     </transmission>
@@ -269,9 +269,9 @@
       <type>transmission_interface/SimpleTransmission</type>
       <joint name="${arm_id}_joint5">
-	<hardwareInterface>hardware_interface/EffortJointInterface</hardwareInterface>
+        <hardwareInterface>hardware_interface/EffortJointInterface</hardwareInterface>
       </joint>
       <actuator name="motor5">
-	<hardwareInterface>hardware_interface/EffortJointInterface</hardwareInterface>
-	<mechanicalReduction>1</mechanicalReduction>
+        <hardwareInterface>hardware_interface/EffortJointInterface</hardwareInterface>
+        <mechanicalReduction>1</mechanicalReduction>
       </actuator>
     </transmission>
@@ -279,9 +279,9 @@
       <type>transmission_interface/SimpleTransmission</type>
       <joint name="${arm_id}_joint6">
-	<hardwareInterface>hardware_interface/EffortJointInterface</hardwareInterface>
+        <hardwareInterface>hardware_interface/EffortJointInterface</hardwareInterface>
       </joint>
       <actuator name="motor6">
-	<hardwareInterface>hardware_interface/EffortJointInterface</hardwareInterface>
-	<mechanicalReduction>1</mechanicalReduction>
+        <hardwareInterface>hardware_interface/EffortJointInterface</hardwareInterface>
+        <mechanicalReduction>1</mechanicalReduction>
       </actuator>
     </transmission>
@@ -289,9 +289,9 @@
       <type>transmission_interface/SimpleTransmission</type>
       <joint name="${arm_id}_joint7">
-	<hardwareInterface>hardware_interface/EffortJointInterface</hardwareInterface>
+        <hardwareInterface>hardware_interface/EffortJointInterface</hardwareInterface>
       </joint>
       <actuator name="motor7">
-	<hardwareInterface>hardware_interface/EffortJointInterface</hardwareInterface>
-	<mechanicalReduction>1</mechanicalReduction>
+        <hardwareInterface>hardware_interface/EffortJointInterface</hardwareInterface>
+        <mechanicalReduction>1</mechanicalReduction>
       </actuator>
     </transmission>

File: ros_ws/src/desc/franka_description/robots/panda_arm_hand_active_vision.xacro (robot description, xacro)
@@ -2,5 +2,5 @@
 <robot xmlns:xacro="http://www.ros.org/wiki/xacro" name="panda">
   <xacro:include filename="$(find franka_description)/robots/panda_arm_active_vision.xacro"/>
-  <xacro:include filename="$(find franka_description)/robots/hand_lockkey.xacro"/>
+  <xacro:include filename="$(find franka_description)/robots/hand_active_vision.xacro"/>
   <xacro:panda_arm />
   <xacro:hand ns="panda" rpy="0 0 ${-pi/4}" connected_to="panda_link8"/>
