Commit message: Show EE in robot description

File: ros_ws/src/desc/franka_description/robots/hand_lockkey.xacro (robot description, xacro)
@@ -59,4 +59,16 @@
         </inertial>
     </link>
+    <!-- <link name="${ns}_end_effector">
+      <visual>
+        <origin xyz="0 0 0.1034" rpy="0 0 0"/>
+      </visual>
+      <collision>
+        <origin xyz="0 0 0" rpy="0 0 ${pi}"/>
+      </collision>
+	<inertial>
+            <mass value="0.1" />
+            <inertia ixx="0.03" iyy="0.03" izz="0.03" ixy="0.0" ixz="0.0" iyz="0.0" />
+        </inertial>
+    </link> -->
   <gazebo reference="panda_leftfinger">
     <kp>1000000.0</kp>
@@ -106,4 +118,8 @@
       <mimic joint="${ns}_finger_joint1" />
     </joint>
+    <!-- <joint name="${ns}_ee_fixed" type="fixed">
+      <parent link="${ns}_hand"/>
+      <child link="${ns}_end_effector"/>
+    </joint> -->
     <transmission name="f_t_1">
       <type>transmission_interface/SimpleTransmission</type>

File: ros_ws/src/desc/franka_description/robots/panda_arm_lockkey.xacro (robot description, xacro)
@@ -224,4 +224,11 @@
       <axis xyz="0 0 0"/>
     </joint>
+    <link name="${arm_id}_EE_control"/>
+    <joint name="${arm_id}_joint8" type="fixed">
+      <origin rpy="0 0 0" xyz="0 0 0.1034"/>
+      <parent link="${arm_id}_link8"/>
+      <child link="${arm_id}_EE_control"/>
+      <axis xyz="0 0 0"/>
+    </joint>
     <!-- Transmissions of the robot arm - to be able to move each joint ============== -->
     <transmission name="tran1">
