Commit message: Added friction and damping

File: ros_ws/src/desc/franka_description/robots/hand.xacro (robot description, xacro)
@@ -36,13 +36,4 @@
         </geometry>
       </collision>
-      <!-- Added friction tag to finger -->
-      <surface>
-        <friction>
-          <ode>
-            <mu>0.7</mu>
-            <mu2>0.7</mu2>
-          </ode>
-        </friction>
-      </surface>
 	<inertial>
             <mass value="0.1" />
@@ -63,13 +54,4 @@
         </geometry>
       </collision>
-      <!-- Added friction tag to finger -->
-      <surface>
-        <friction>
-          <ode>
-            <mu>0.7</mu>
-            <mu2>0.7</mu2>
-          </ode>
-        </friction>
-      </surface>
 	<inertial>
             <mass value="0.1" />
@@ -77,4 +59,18 @@
         </inertial>
     </link>
+  <gazebo reference="panda_leftfinger">
+    <kp>1000000.0</kp>
+    <kd>1.0</kd>
+    <mu1>1.0</mu1>
+    <mu2>1.0</mu2>
+    <minDepth>0.001</minDepth>
+  </gazebo>
+  <gazebo reference="panda_rightfinger">
+    <kp>1000000.0</kp>
+    <kd>1.0</kd>
+    <mu1>1.0</mu1>
+    <mu2>1.0</mu2>
+    <minDepth>0.001</minDepth>
+  </gazebo>
     <joint name="${ns}_finger_joint1" type="prismatic">
       <parent link="${ns}_hand"/>
@@ -82,5 +78,5 @@
       <origin xyz="0 0 0.0584" rpy="0 0 0"/>
       <axis xyz="0 1 0"/>
-      <limit effort="20" lower="0.0" upper="0.04" velocity="0.2"/>
+      <limit effort="50" lower="0.0" upper="0.04" velocity="0.2"/>
     </joint>
     <joint name="${ns}_finger_joint2" type="prismatic">
@@ -89,5 +85,5 @@
       <origin xyz="0 0 0.0584" rpy="0 0 0"/>
       <axis xyz="0 -1 0"/>
-      <limit effort="20" lower="0.0" upper="0.04" velocity="0.2"/>
+      <limit effort="50" lower="0.0" upper="0.04" velocity="0.1"/>
       <mimic joint="${ns}_finger_joint1" />
     </joint>

Commit message: decreased max vel for fingers

File: ros_ws/src/desc/franka_description/robots/hand.xacro (robot description, xacro)
@@ -78,5 +78,5 @@
       <origin xyz="0 0 0.0584" rpy="0 0 0"/>
       <axis xyz="0 1 0"/>
-      <limit effort="50" lower="0.0" upper="0.04" velocity="0.2"/>
+      <limit effort="50" lower="0.0" upper="0.04" velocity="0.1"/>
     </joint>
     <joint name="${ns}_finger_joint2" type="prismatic">

Commit message: tuned friction

File: ros_ws/src/desc/franka_description/robots/hand.xacro (robot description, xacro)
@@ -62,6 +62,6 @@
     <kp>1000000.0</kp>
     <kd>1.0</kd>
-    <mu1>1.0</mu1>
-    <mu2>1.0</mu2>
+    <mu1>100000.0</mu1>
+    <mu2>100000.0</mu2>
     <minDepth>0.001</minDepth>
   </gazebo>
@@ -69,6 +69,6 @@
     <kp>1000000.0</kp>
     <kd>1.0</kd>
-    <mu1>1.0</mu1>
-    <mu2>1.0</mu2>
+    <mu1>100000.0</mu1>
+    <mu2>100000.0</mu2>
     <minDepth>0.001</minDepth>
   </gazebo>
@@ -78,5 +78,5 @@
       <origin xyz="0 0 0.0584" rpy="0 0 0"/>
       <axis xyz="0 1 0"/>
-      <limit effort="50" lower="0.0" upper="0.04" velocity="0.1"/>
+      <limit effort="1000" lower="0.0" upper="0.04" velocity="0.1"/>
     </joint>
     <joint name="${ns}_finger_joint2" type="prismatic">
@@ -85,5 +85,5 @@
       <origin xyz="0 0 0.0584" rpy="0 0 0"/>
       <axis xyz="0 -1 0"/>
-      <limit effort="50" lower="0.0" upper="0.04" velocity="0.1"/>
+      <limit effort="1000" lower="0.0" upper="0.04" velocity="0.1"/>
       <mimic joint="${ns}_finger_joint1" />
     </joint>

Commit message: Integrating with lab PC files

File: ros_ws/src/desc/franka_description/robots/hand.xacro (robot description, xacro)
@@ -1,5 +1,6 @@
 <?xml version="1.0" encoding="utf-8"?>
 <robot xmlns:xacro="http://www.ros.org/wiki/xacro" name="hand">
-  <xacro:macro name="hand" params="connected_to:='' ns:='' rpy:='0 0 0' xyz:='0 0 0' ">
+  <!-- safety_distance: Minimum safety distance in [m] by which the collision volumes are expanded and which is enforced during robot motions -->
+  <xacro:macro name="hand" params="connected_to:='' ns:='' rpy:='0 0 0' xyz:='0 0 0' safety_distance:=0">
     <xacro:unless value="${connected_to == ''}">
       <joint name="${ns}_hand_joint" type="fixed">
@@ -16,12 +17,43 @@
       </visual>
       <collision>
+        <origin xyz="0 0 0.04" rpy="0 ${pi/2} ${pi/2}"/>
         <geometry>
-          <mesh filename="package://franka_description/meshes/collision/hand.stl"/>
+          <cylinder radius="${0.04+safety_distance}" length="0.1" />
         </geometry>
       </collision>
-	<inertial>
-            <mass value="0.1" />
-            <inertia ixx="0.03" iyy="0.03" izz="0.03" ixy="0.0" ixz="0.0" iyz="0.0" />
-        </inertial>
+      <collision>
+        <origin xyz="0 -0.05 0.04" rpy="0 0 0"/>
+        <geometry>
+          <sphere radius="${0.04+safety_distance}"  />
+        </geometry>
+      </collision>
+      <collision>
+        <origin xyz="0 0.05 0.04" rpy="0 0 0"/>
+        <geometry>
+          <sphere radius="${0.04+safety_distance}"  />
+        </geometry>
+      </collision>
+      <collision>
+        <origin xyz="0 0 0.1" rpy="0 ${pi/2} ${pi/2}"/>
+        <geometry>
+          <cylinder radius="${0.02+safety_distance}" length="0.1" />
+        </geometry>
+      </collision>
+      <collision>
+        <origin xyz="0 -0.05 0.1" rpy="0 0 0"/>
+        <geometry>
+          <sphere radius="${0.02+safety_distance}"  />
+        </geometry>
+      </collision>
+      <collision>
+        <origin xyz="0 0.05 0.1" rpy="0 0 0"/>
+        <geometry>
+          <sphere radius="${0.02+safety_distance}"  />
+        </geometry>
+      </collision>
+      <inertial>
+        <mass value="0.1" />
+        <inertia ixx="0.03" iyy="0.03" izz="0.03" ixy="0.0" ixz="0.0" iyz="0.0" />
+      </inertial>
     </link>
     <link name="${ns}_leftfinger">
@@ -31,13 +63,8 @@
         </geometry>
       </visual>
-      <collision>
-        <geometry>
-          <mesh filename="package://franka_description/meshes/collision/finger.stl"/>
-        </geometry>
-      </collision>
-	<inertial>
-            <mass value="0.1" />
-            <inertia ixx="0.03" iyy="0.03" izz="0.03" ixy="0.0" ixz="0.0" iyz="0.0" />
-        </inertial>
+      <inertial>
+        <mass value="0.1" />
+        <inertia ixx="0.03" iyy="0.03" izz="0.03" ixy="0.0" ixz="0.0" iyz="0.0" />
+      </inertial>
     </link>
     <link name="${ns}_rightfinger">
@@ -48,29 +75,9 @@
         </geometry>
       </visual>
-      <collision>
-        <origin xyz="0 0 0" rpy="0 0 ${pi}"/>
-        <geometry>
-          <mesh filename="package://franka_description/meshes/collision/finger.stl"/>
-        </geometry>
-      </collision>
-	<inertial>
-            <mass value="0.1" />
-            <inertia ixx="0.03" iyy="0.03" izz="0.03" ixy="0.0" ixz="0.0" iyz="0.0" />
-        </inertial>
-    </link>
-  <gazebo reference="panda_leftfinger">
-    <kp>1000000.0</kp>
-    <kd>1.0</kd>
-    <mu1>100000.0</mu1>
-    <mu2>100000.0</mu2>
-    <minDepth>0.001</minDepth>
-  </gazebo>
-  <gazebo reference="panda_rightfinger">
-    <kp>1000000.0</kp>
-    <kd>1.0</kd>
-    <mu1>100000.0</mu1>
-    <mu2>100000.0</mu2>
-    <minDepth>0.001</minDepth>
-  </gazebo>
+      <inertial>
+        <mass value="0.1" />
+        <inertia ixx="0.03" iyy="0.03" izz="0.03" ixy="0.0" ixz="0.0" iyz="0.0" />
+      </inertial>
+   </link>
     <joint name="${ns}_finger_joint1" type="prismatic">
       <parent link="${ns}_hand"/>
@@ -78,5 +85,5 @@
       <origin xyz="0 0 0.0584" rpy="0 0 0"/>
       <axis xyz="0 1 0"/>
-      <limit effort="1000" lower="0.0" upper="0.04" velocity="0.1"/>
+      <limit effort="20" lower="0.0" upper="0.04" velocity="0.2"/>
     </joint>
     <joint name="${ns}_finger_joint2" type="prismatic">
@@ -85,27 +92,7 @@
       <origin xyz="0 0 0.0584" rpy="0 0 0"/>
       <axis xyz="0 -1 0"/>
-      <limit effort="1000" lower="0.0" upper="0.04" velocity="0.1"/>
+      <limit effort="20" lower="0.0" upper="0.04" velocity="0.2"/>
       <mimic joint="${ns}_finger_joint1" />
     </joint>
-    <transmission name="f_t_1">
-      <type>transmission_interface/SimpleTransmission</type>
-      <joint name="${ns}_finger_joint1">
-	<hardwareInterface>hardware_interface/EffortJointInterface</hardwareInterface>
-      </joint>
-      <actuator name="motor_finger_1">
-	<hardwareInterface>hardware_interface/EffortJointInterface</hardwareInterface>
-	<mechanicalReduction>1</mechanicalReduction>
-      </actuator>
-    </transmission>
-    <transmission name="f_t_2">
-      <type>transmission_interface/SimpleTransmission</type>
-      <joint name="${ns}_finger_joint2">
-	<hardwareInterface>hardware_interface/EffortJointInterface</hardwareInterface>
-      </joint>
-      <actuator name="motor_finger_2">
-	<hardwareInterface>hardware_interface/EffortJointInterface</hardwareInterface>
-	<mechanicalReduction>1</mechanicalReduction>
-      </actuator>
-    </transmission>
   </xacro:macro>
 </robot>

File: ros_ws/src/desc/franka_description/robots/panda_arm.xacro (robot description, xacro)
@@ -1,5 +1,7 @@
 <?xml version='1.0' encoding='utf-8'?>
 <robot xmlns:xacro="http://www.ros.org/wiki/xacro" name="panda">
-  <xacro:macro name="panda_arm" params="arm_id:='panda' description_pkg:='franka_description' connected_to:='' xyz:='0 0 0' rpy:='0 0 0'">
+  <!-- safety_distance: Minimum safety distance in [m] by which the collision volumes are expanded and which is enforced during robot motions -->
+  <!-- arm_id: Namespace of the panda arm. Serves to differentiate between arms in case of multiple instances. -->
+  <xacro:macro name="panda_arm" params="arm_id:='panda' description_pkg:='franka_description' connected_to:='' xyz:='0 0 0' rpy:='0 0 0' safety_distance:=0">
     <xacro:unless value="${not connected_to}">
       <joint name="${arm_id}_joint_${connected_to}" type="fixed">
@@ -9,9 +11,4 @@
       </joint>
     </xacro:unless>
-    <link name="world"/>
-    <joint name="fixed" type="fixed">
-      <parent link="world"/>
-      <child link="${arm_id}_link0"/>
-    </joint>
     <link name="${arm_id}_link0">
       <visual>
@@ -21,12 +18,21 @@
       </visual>
       <collision>
-        <geometry>
-          <mesh filename="package://${description_pkg}/meshes/collision/link0.stl"/>
-        </geometry>
-      </collision>
-      <inertial>
-        <mass value="0.1" />
-        <inertia ixx="0.03" iyy="0.03" izz="0.03" ixy="0.0" ixz="0.0" iyz="0.0" />
-      </inertial>
+        <origin xyz="-0.075 0 0.06" rpy="0 ${pi/2} 0"/>
+        <geometry>
+          <cylinder radius="${0.06+safety_distance}" length="0.03" />
+        </geometry>
+      </collision>
+      <collision>
+        <origin xyz="-0.06 0 0.06" rpy="0 0 0"/>
+        <geometry>
+          <sphere radius="${0.06+safety_distance}" />
+        </geometry>
+      </collision>
+      <collision>
+        <origin xyz="-0.09 0 0.06" rpy="0 0 0"/>
+        <geometry>
+          <sphere radius="${0.06+safety_distance}" />
+        </geometry>
+      </collision>
     </link>
     <link name="${arm_id}_link1">
@@ -37,12 +43,21 @@
       </visual>
       <collision>
-        <geometry>
-          <mesh filename="package://${description_pkg}/meshes/collision/link1.stl"/>
-        </geometry>
-      </collision>
-      <inertial>
-        <mass value="0.1" />
-        <inertia ixx="0.03" iyy="0.03" izz="0.03" ixy="0.0" ixz="0.0" iyz="0.0" />
-      </inertial>
+        <origin xyz="0 0 -0.1915" rpy="0 0 0"/>
+        <geometry>
+          <cylinder radius="${0.06+safety_distance}" length="0.2830" />
+        </geometry>
+      </collision>
+      <collision>
+        <origin xyz="0 0 -0.333" rpy="0 0 0"/>
+        <geometry>
+          <sphere radius="${0.06+safety_distance}" />
+        </geometry>
+      </collision>
+      <collision>
+        <origin xyz="0 0 -0.05" rpy="0 0 0"/>
+        <geometry>
+          <sphere radius="${0.06+safety_distance}" />
+        </geometry>
+      </collision>
     </link>
     <joint name="${arm_id}_joint1" type="revolute">
@@ -61,12 +76,21 @@
       </visual>
       <collision>
-        <geometry>
-          <mesh filename="package://${description_pkg}/meshes/collision/link2.stl"/>
-        </geometry>
-      </collision>
-      <inertial>
-        <mass value="0.1" />
-        <inertia ixx="0.03" iyy="0.03" izz="0.03" ixy="0.0" ixz="0.0" iyz="0.0" />
-      </inertial>
+        <origin xyz="0 0 0" rpy="0 0 0"/>
+        <geometry>
+          <cylinder radius="${0.06+safety_distance}" length="0.12" />
+        </geometry>
+      </collision>
+      <collision>
+        <origin xyz="0 0 -0.06" rpy="0 0 0"/>
+        <geometry>
+          <sphere radius="${0.06+safety_distance}" />
+        </geometry>
+      </collision>
+      <collision>
+        <origin xyz="0 0 0.06" rpy="0 0 0"/>
+        <geometry>
+          <sphere radius="${0.06+safety_distance}" />
+        </geometry>
+      </collision>
     </link>
     <joint name="${arm_id}_joint2" type="revolute">
@@ -85,12 +109,21 @@
       </visual>
       <collision>
-        <geometry>
-          <mesh filename="package://${description_pkg}/meshes/collision/link3.stl"/>
-        </geometry>
-      </collision>
-      <inertial>
-        <mass value="0.1" />
-        <inertia ixx="0.03" iyy="0.03" izz="0.03" ixy="0.0" ixz="0.0" iyz="0.0" />
-      </inertial>
+        <origin xyz="0 0 -0.145" rpy="0 0 0"/>
+        <geometry>
+          <cylinder radius="${0.06+safety_distance}" length="0.15" />
+        </geometry>
+      </collision>
+      <collision>
+        <origin xyz="0 0 -0.22" rpy="0 0 0"/>
+        <geometry>
+          <sphere radius="${0.06+safety_distance}" />
+        </geometry>
+      </collision>
+      <collision>
+        <origin xyz="0 0 -0.07" rpy="0 0 0"/>
+        <geometry>
+          <sphere radius="${0.06+safety_distance}" />
+        </geometry>
+      </collision>
     </link>
     <joint name="${arm_id}_joint3" type="revolute">
@@ -109,12 +142,21 @@
       </visual>
       <collision>
-        <geometry>
-          <mesh filename="package://${description_pkg}/meshes/collision/link4.stl"/>
-        </geometry>
-      </collision>
-      <inertial>
-        <mass value="0.1" />
-        <inertia ixx="0.03" iyy="0.03" izz="0.03" ixy="0.0" ixz="0.0" iyz="0.0" />
-      </inertial>
+        <origin xyz="0 0 0" rpy="0 0 0"/>
+        <geometry>
+          <cylinder radius="${0.06+safety_distance}" length="0.12" />
+        </geometry>
+      </collision>
+      <collision>
+        <origin xyz="0 0 0.06" rpy="0 0 0"/>
+        <geometry>
+          <sphere radius="${0.06+safety_distance}" />
+        </geometry>
+      </collision>
+      <collision>
+        <origin xyz="0 0 -0.06" rpy="0 0 0"/>
+        <geometry>
+          <sphere radius="${0.06+safety_distance}" />
+        </geometry>
+      </collision>
     </link>
     <joint name="${arm_id}_joint4" type="revolute">
@@ -133,12 +175,39 @@
       </visual>
       <collision>
-        <geometry>
-          <mesh filename="package://${description_pkg}/meshes/collision/link5.stl"/>
-        </geometry>
-      </collision>
-      <inertial>
-        <mass value="0.1" />
-        <inertia ixx="0.03" iyy="0.03" izz="0.03" ixy="0.0" ixz="0.0" iyz="0.0" />
-      </inertial>
+        <origin xyz="0 0 -0.26" rpy="0 0 0"/>
+        <geometry>
+          <cylinder radius="${0.06+safety_distance}" length="0.1" />
+        </geometry>
+      </collision>
+      <collision>
+        <origin xyz="0 0 -0.31" rpy="0 0 0"/>
+        <geometry>
+          <sphere radius="${0.06+safety_distance}" />
+        </geometry>
+      </collision>
+      <collision>
+        <origin xyz="0 0 -0.21" rpy="0 0 0"/>
+        <geometry>
+          <sphere radius="${0.06+safety_distance}" />
+        </geometry>
+      </collision>
+      <collision>
+        <origin xyz="0 0.08 -0.13" rpy="0 0 0"/>
+        <geometry>
+          <cylinder radius="${0.025+safety_distance}" length="0.14" />
+        </geometry>
+      </collision>
+      <collision>
+        <origin xyz="0 0.08 -0.06" rpy="0 0 0"/>
+        <geometry>
+          <sphere radius="${0.025+safety_distance}" />
+        </geometry>
+      </collision>
+      <collision>
+        <origin xyz="0 0.08 -0.20" rpy="0 0 0"/>
+        <geometry>
+          <sphere radius="${0.025+safety_distance}" />
+        </geometry>
+      </collision>
     </link>
     <joint name="${arm_id}_joint5" type="revolute">
@@ -157,12 +226,21 @@
       </visual>
       <collision>
-        <geometry>
-          <mesh filename="package://${description_pkg}/meshes/collision/link6.stl"/>
-        </geometry>
-      </collision>
-      <inertial>
-        <mass value="0.1" />
-        <inertia ixx="0.03" iyy="0.03" izz="0.03" ixy="0.0" ixz="0.0" iyz="0.0" />
-      </inertial>
+        <origin xyz="0 0 -0.03" rpy="0 0 0"/>
+        <geometry>
+          <cylinder radius="${0.05+safety_distance}" length="0.08" />
+        </geometry>
+      </collision>
+      <collision>
+        <origin xyz="0 0 0.01" rpy="0 0 0"/>
+        <geometry>
+          <sphere radius="${0.05+safety_distance}" />
+        </geometry>
+      </collision>
+      <collision>
+        <origin xyz="0 0 -0.07" rpy="0 0 0"/>
+        <geometry>
+          <sphere radius="${0.05+safety_distance}" />
+        </geometry>
+      </collision>
     </link>
     <joint name="${arm_id}_joint6" type="revolute">
@@ -181,12 +259,21 @@
       </visual>
       <collision>
-        <geometry>
-          <mesh filename="package://${description_pkg}/meshes/collision/link7.stl"/>
-        </geometry>
-      </collision>
-      <inertial>
-        <mass value="0.1" />
-        <inertia ixx="0.03" iyy="0.03" izz="0.03" ixy="0.0" ixz="0.0" iyz="0.0" />
-      </inertial>
+        <origin xyz="0 0 0.01" rpy="0 0 0"/>
+        <geometry>
+          <cylinder radius="${0.04+safety_distance}" length="0.14" />
+        </geometry>
+      </collision>
+      <collision>
+        <origin xyz="0 0 0.08" rpy="0 0 0"/>
+        <geometry>
+          <sphere radius="${0.04+safety_distance}"  />
+        </geometry>
+      </collision>
+      <collision>
+        <origin xyz="0 0 -0.06" rpy="0 0 0"/>
+        <geometry>
+          <sphere radius="${0.04+safety_distance}"  />
+        </geometry>
+      </collision>
     </link>
     <joint name="${arm_id}_joint7" type="revolute">
@@ -198,89 +285,29 @@
       <limit effort="12" lower="-2.8973" upper="2.8973" velocity="2.6100"/>
     </joint>
-    <link name="${arm_id}_link8"/>
+    <link name="${arm_id}_link8">
+      <collision>
+        <origin xyz="0.0424 0.0424 -0.0250" rpy="${pi} ${pi/2} ${pi/2}"/>
+        <geometry>
+          <cylinder radius="${0.03+safety_distance}"  length="0.01" />
+        </geometry>
+      </collision>
+      <collision>
+        <origin xyz="0.0424 0.0424 -0.02" rpy="0 0 0"/>
+        <geometry>
+          <sphere radius="${0.03+safety_distance}"  />
+        </geometry>
+      </collision>
+      <collision>
+        <origin xyz="0.0424 0.0424 -0.03" rpy="0 0 0"/>
+        <geometry>
+          <sphere radius="${0.03+safety_distance}"  />
+        </geometry>
+      </collision>
+    </link>
     <joint name="${arm_id}_joint8" type="fixed">
       <origin rpy="0 0 0" xyz="0 0 0.107"/>
       <parent link="${arm_id}_link7"/>
       <child link="${arm_id}_link8"/>
-      <axis xyz="0 0 0"/>
-    </joint>
-    <!-- Transmissions of the robot arm - to be able to move each joint ============== -->
-    <transmission name="tran1">
-      <type>transmission_interface/SimpleTransmission</type>
-      <joint name="${arm_id}_joint1">
-	<hardwareInterface>hardware_interface/EffortJointInterface</hardwareInterface>
-      </joint>
-      <actuator name="motor1">
-	<hardwareInterface>hardware_interface/EffortJointInterface</hardwareInterface>
-	<mechanicalReduction>1</mechanicalReduction>
-      </actuator>
-    </transmission>
-    <transmission name="tran2">
-      <type>transmission_interface/SimpleTransmission</type>
-      <joint name="${arm_id}_joint2">
-	<hardwareInterface>hardware_interface/EffortJointInterface</hardwareInterface>
-      </joint>
-      <actuator name="motor2">
-	<hardwareInterface>hardware_interface/EffortJointInterface</hardwareInterface>
-	<mechanicalReduction>1</mechanicalReduction>
-      </actuator>
-    </transmission>
-    <transmission name="tran3">
-      <type>transmission_interface/SimpleTransmission</type>
-      <joint name="${arm_id}_joint3">
-	<hardwareInterface>hardware_interface/EffortJointInterface</hardwareInterface>
-      </joint>
-      <actuator name="motor3">
-	<hardwareInterface>hardware_interface/EffortJointInterface</hardwareInterface>
-	<mechanicalReduction>1</mechanicalReduction>
-      </actuator>
-    </transmission>
-    <transmission name="tran4">
-      <type>transmission_interface/SimpleTransmission</type>
-      <joint name="${arm_id}_joint4">
-	<hardwareInterface>hardware_interface/EffortJointInterface</hardwareInterface>
-      </joint>
-      <actuator name="motor4">
-	<hardwareInterface>hardware_interface/EffortJointInterface</hardwareInterface>
-	<mechanicalReduction>1</mechanicalReduction>
-      </actuator>
-    </transmission>
-    <transmission name="tran5">
-      <type>transmission_interface/SimpleTransmission</type>
-      <joint name="${arm_id}_joint5">
-	<hardwareInterface>hardware_interface/EffortJointInterface</hardwareInterface>
-      </joint>
-      <actuator name="motor5">
-	<hardwareInterface>hardware_interface/EffortJointInterface</hardwareInterface>
-	<mechanicalReduction>1</mechanicalReduction>
-      </actuator>
-    </transmission>
-    <transmission name="tran6">
-      <type>transmission_interface/SimpleTransmission</type>
-      <joint name="${arm_id}_joint6">
-	<hardwareInterface>hardware_interface/EffortJointInterface</hardwareInterface>
-      </joint>
-      <actuator name="motor6">
-	<hardwareInterface>hardware_interface/EffortJointInterface</hardwareInterface>
-	<mechanicalReduction>1</mechanicalReduction>
-      </actuator>
-    </transmission>
-    <transmission name="tran7">
-      <type>transmission_interface/SimpleTransmission</type>
-      <joint name="${arm_id}_joint7">
-	<hardwareInterface>hardware_interface/EffortJointInterface</hardwareInterface>
-      </joint>
-      <actuator name="motor7">
-	<hardwareInterface>hardware_interface/EffortJointInterface</hardwareInterface>
-	<mechanicalReduction>1</mechanicalReduction>
-      </actuator>
-    </transmission>
+    </joint>
   </xacro:macro>
-  <!-- Gazebo control plugin -->
-  <gazebo>
-    <plugin name="gazebo_ros_control" filename="libgazebo_ros_control.so">
-      <robotNamespace>/panda</robotNamespace>
-      <robotSimType>gazebo_ros_control/DefaultRobotHWSim</robotSimType>
-    </plugin>
-  </gazebo>
 </robot>
