Commit message: Ignoring grasps not reachable by franka

File: ros_ws/src/desc/franka_description/robots/hand_active_vision.xacro (robot description, xacro)
@@ -13,4 +13,10 @@
         <geometry>
           <mesh filename="package://franka_description/meshes/visual/hand.dae"/>
+        </geometry>
+      </visual>
+      <visual>
+        <origin xyz="0.05 0.0 0.05" rpy="-${pi/2} -${pi/2} -${pi/2}"/>
+        <geometry>
+          <mesh filename="package://active_vision/models/kinectAV/meshes/kinect.dae"/>
         </geometry>
       </visual>

File: ros_ws/src/projects/active_vision/desc/franka_camera.xacro (robot description, xacro)
@@ -12,4 +12,4 @@
   </joint>
   <!-- <xacro:camera_gazebo_sensor xyz="0.05 -0.05 0" rpy="-1.57 -1.57 -0.785" parent="panda_link8" sensor_name="camera"/> -->
-  <xacro:camera_gazebo_sensor xyz="0.06 0 0" rpy="-1.57 -1.57 -1.57" parent="panda_hand" sensor_name="camera"/>
+  <xacro:camera_gazebo_sensor xyz="0.05 0 0.05" rpy="-1.57 -1.57 -1.57" parent="panda_hand" sensor_name="camera"/>
 </robot>

Commit message: Adding visibility constraints

File: ros_ws/src/desc/franka_description/robots/hand_active_vision.xacro (robot description, xacro)
@@ -18,5 +18,5 @@
         <origin xyz="0.05 0.0 0.05" rpy="-${pi/2} -${pi/2} -${pi/2}"/>
         <geometry>
-          <mesh filename="package://active_vision/models/kinectAV/meshes/kinect.dae"/>
+          <mesh filename="package://active_vision/models/kinectAV/meshes/realsense.stl"/>
         </geometry>
       </visual>

Commit message: realsense offset update

File: ros_ws/src/desc/franka_description/robots/hand_active_vision.xacro (robot description, xacro)
@@ -16,7 +16,13 @@
       </visual>
       <visual>
-        <origin xyz="0.05 0.0 0.05" rpy="-${pi/2} -${pi/2} -${pi/2}"/>
+        <origin xyz="0.03 0.0 0.07" rpy="-${pi/2} -${pi/2} -${pi/2}"/>
         <geometry>
           <mesh filename="package://active_vision/models/kinectAV/meshes/realsense.stl"/>
+        </geometry>
+      </visual>
+      <visual>
+        <origin xyz="0.018 0.0 0.007" rpy="0 0 0"/>
+        <geometry>
+          <mesh filename="package://active_vision/models/kinectAV/meshes/panda_realsenseD435_mount.stl"/>
         </geometry>
       </visual>

File: ros_ws/src/projects/active_vision/desc/franka_camera.xacro (robot description, xacro)
@@ -12,4 +12,4 @@
   </joint>
   <!-- <xacro:camera_gazebo_sensor xyz="0.05 -0.05 0" rpy="-1.57 -1.57 -0.785" parent="panda_link8" sensor_name="camera"/> -->
-  <xacro:camera_gazebo_sensor xyz="0.05 0 0.05" rpy="-1.57 -1.57 -1.57" parent="panda_hand" sensor_name="camera"/>
+  <xacro:camera_gazebo_sensor xyz="0.03 0.0175 0.07" rpy="-1.57 -1.57 -1.57" parent="panda_hand" sensor_name="camera"/>
 </robot>
