Commit message: Added wooden block, despawner

File: ros_ws/src/projects/table_rearrange/ycb_models/desc/wood_block.urdf (robot description, URDF)
Before this commit: robot mug, 2 links, 1 joints
Links:
- removed link mug
- added link wood_block, mass 0.01; collision mesh filename=package://ycb_models/mesh/wood_block/textured.dae; visual mesh filename=package://ycb_models/mesh/wood_block/textured.dae
Joints:
- removed joint table_mug
- added joint table_wood_block: type floating, parent world, child wood_block, origin xyz=0 0 0 rpy=0 0 0
