Commit message: Moved files, added items to YCB

File: ros_ws/src/projects/table_rearrange/ycb_models/desc/master_chef_can.urdf (robot description, URDF)
Before this commit: robot master_chef_can, 2 links, 1 joints
Links:
- link master_chef_can: mass 0.001088 -> 0.001; geometry collision mesh filename=package://ycb_models/mesh/master_chef_can/textured.dae; visual mesh filename=package://ycb_models/mesh/master_chef_can/textured.dae
