Commit message: Added extra conveyor objects, fixed textures

File: ros_ws/src/projects/table_rearrange/ycb_models/desc/mug.urdf (robot description, URDF)
Before this commit: robot mug, 2 links, 1 joints
Links:
- link mug: geometry collision mesh filename=package://ycb_models/mesh/mug/textured.dae; visual mesh filename=package://ycb_models/mesh/mug/textured.dae
