Commit message: simulation parameter updates

File: ros_ws/src/desc/vf-hand_description/robots/vf_hand.urdf (robot description, URDF)
Before this commit: robot vf_hand, 4 links, 3 joints
Joints:
- joint J1: limit lower=0 upper=0 effort=10 velocity=0.5 -> lower=-0.8 upper=0.8 effort=1 velocity=0.5
- joint J2: limit lower=0 upper=0 effort=10 velocity=0.5 -> lower=-0.8 upper=0.8 effort=1 velocity=0.5
