Commit message: simulation glitches fixed

File: ros_ws/src/desc/vf-hand_description/robots/vf_hand.xacro (robot description, xacro)
@@ -108,8 +108,8 @@
     <axis
       xyz="1 0 0" />
-    <!-- <dynamics damping="1.0" friction="10.0"/> -->
+    <dynamics damping="0.01" friction="0.01"/>
     <limit
-      lower="0"
-      upper="0"
+      lower="-0.8"
+      upper="0.8"
       effort="1"
       velocity="0.5" />
@@ -169,8 +169,8 @@
     <axis
       xyz="1 0 0" />
-    <!-- <dynamics damping="1.0" friction="10.0"/> -->
+    <dynamics damping="0.01" friction="0.01"/>
     <limit
-      lower="0"
-      upper="0"
+      lower="-0.8"
+      upper="0.8"
       effort="1"
       velocity="0.5" />
