Commit message: Setup conveyor belt

File: ros_ws/src/projects/table_rearrange/table_rearrange/desc/table_surface.urdf (robot description, URDF)
Before this commit: robot table_surface, 2 links, 1 joints
Links:
- link table: geometry collision box size=2 2 0.05; visual box size=2 2 0.05
Joints:
- joint fixed: origin xyz=0.5 0 0.25 rpy=0 0 0 -> xyz=1.1 0 0.05 rpy=0 0 0
