Commit message: relaxedik setup

File: ros_ws/src/relaxed_ik/src/RelaxedIK/urdfs/updated_panda_arm.xacro (robot description, xacro)
@@ -281,18 +281,18 @@
     <minDepth>0.001</minDepth>
   </gazebo>
-    <joint name="panda_finger_joint1" type="prismatic">
+    <joint name="panda_finger_joint1" type="fixed">
       <parent link="panda_hand"/>
       <child link="panda_leftfinger"/>
       <origin xyz="0 0 0.0584" rpy="0 0 0"/>
       <axis xyz="0 1 0"/>
-      <limit effort="1000" lower="0.0" upper="0.04" velocity="0.1"/>
-    </joint>
-    <joint name="panda_finger_joint2" type="prismatic">
+      <!-- <limit effort="1000" lower="0.0" upper="0.04" velocity="0.1"/> -->
+    </joint>
+    <joint name="panda_finger_joint2" type="fixed">
       <parent link="panda_hand"/>
       <child link="panda_rightfinger"/>
       <origin xyz="0 0 0.0584" rpy="0 0 0"/>
       <axis xyz="0 -1 0"/>
-      <limit effort="1000" lower="0.0" upper="0.04" velocity="0.1"/>
-      <mimic joint="panda_finger_joint1" />
+      <!-- <limit effort="1000" lower="0.0" upper="0.04" velocity="0.1"/>
+      <mimic joint="panda_finger_joint1" /> -->
     </joint>
     <link name="panda_ee_link"/>
@@ -300,4 +300,5 @@
       <parent link="panda_hand"/>
       <child link="panda_ee_link"/>
+      <axis xyz="0 0 0"/>
     </joint>
     <transmission name="f_t_1">
