Commit message: created encoderless folder

File: ros_ws/src/projects/encoderless_robots/desc/updated_hand.xacro (robot description, xacro)
@@ -73,20 +73,20 @@
     <minDepth>0.001</minDepth>
   </gazebo>
-    <joint name="${ns}_finger_joint1" type="prismatic">
+    <joint name="${ns}_finger_joint1" type="fixed">
       <parent link="${ns}_hand"/>
       <child link="${ns}_leftfinger"/>
-      <origin xyz="0 0 0.0584" rpy="0 0 0"/>
+      <origin xyz="0 0.02 0.0584" rpy="0 0 0"/>
       <axis xyz="0 1 0"/>
-      <limit effort="1000" lower="0.0" upper="0.04" velocity="0.1"/>
+      <!-- <limit effort="1000" lower="0.0" upper="0.04" velocity="0.1"/> -->
     </joint>
-    <joint name="${ns}_finger_joint2" type="prismatic">
+    <joint name="${ns}_finger_joint2" type="fixed">
       <parent link="${ns}_hand"/>
       <child link="${ns}_rightfinger"/>
-      <origin xyz="0 0 0.0584" rpy="0 0 0"/>
+      <origin xyz="0 0.02 0.0584" rpy="0 0 0"/>
       <axis xyz="0 -1 0"/>
-      <limit effort="1000" lower="0.0" upper="0.04" velocity="0.1"/>
-      <mimic joint="${ns}_finger_joint1" />
+      <!-- <limit effort="1000" lower="0.0" upper="0.04" velocity="0.1"/>
+      <mimic joint="${ns}_finger_joint1" /> -->
     </joint>
-    <transmission name="f_t_1">
+    <!-- <transmission name="f_t_1">
       <type>transmission_interface/SimpleTransmission</type>
       <joint name="${ns}_finger_joint1">
@@ -107,5 +107,5 @@
 	<mechanicalReduction>1</mechanicalReduction>
       </actuator>
-    </transmission>
+    </transmission> -->
   </xacro:macro>
 </robot>
