Commit message: Added custom Gazebo Hardware Interface

File: ros_ws/src/projects/encoderless_robots/desc/camera_on_stand.xacro (robot description, xacro)
@@ -1,4 +1,4 @@
 <?xml version="1.0" encoding="utf-8"?>
-<robot xmlns:xacro="http://www.ros.org/wiki/xacro" name="green_ball">
+<robot xmlns:xacro="http://www.ros.org/wiki/xacro" name="camera_on_stand">
   <xacro:macro name="camera_on_stand">
     <gazebo reference="camera_link">
@@ -72,5 +72,5 @@
               <origin xyz="0 0 0" rpy="0 0 0"/>
                <geometry>
-                <mesh filename="package://encoderless_robots/meshes/kinect/kinect.dae"/>
+                <mesh filename="package://encoderless_robots/meshes/kinect.dae"/>
                 <!-- <mesh scale="0.005 0.005 0.005" filename="package://vision_control/meshes/tripod/tripod.dae"/> -->
                </geometry>

File: ros_ws/src/projects/encoderless_robots/desc/top_module.xacro (robot description, xacro)
@@ -12,4 +12,12 @@
   <xacro:updated_hand ns="panda" rpy="0 0 0" connected_to="panda_link8"/>
   <xacro:camera_on_stand />
+  <!-- Gazebo control plugin -->
+  <gazebo>
+    <!-- <plugin name="gazebo_ros_control" filename="libmy_gazebo_ros_control.so"> -->
+      <plugin name="gazebo_ros_control" filename="libgazebo_ros_control.so">
+      <robotNamespace>/panda</robotNamespace>
+      <!-- <robotSimType>gazebo_ros_control/DefaultRobotHWSim</robotSimType> -->
+    </plugin>
+  </gazebo>
   <!-- <xacro:hand ns="panda" rpy="0 0 ${-pi/4}" connected_to="panda_link8"/> -->
   <!-- <joint name="panda_hand_joint" type="fixed">

File: ros_ws/src/projects/encoderless_robots/desc/updated_hand.xacro (robot description, xacro)
@@ -83,5 +83,5 @@
       <parent link="${ns}_hand"/>
       <child link="${ns}_rightfinger"/>
-      <origin xyz="0 0.02 0.0584" rpy="0 0 0"/>
+      <origin xyz="0 -0.02 0.0584" rpy="0 0 0"/>
       <axis xyz="0 -1 0"/>
       <!-- <limit effort="1000" lower="0.0" upper="0.04" velocity="0.1"/>

File: ros_ws/src/projects/encoderless_robots/desc/updated_panda_arm.xacro (robot description, xacro)
@@ -277,11 +277,3 @@
     </transmission>
   </xacro:macro>
-  <!-- Gazebo control plugin -->
-  <gazebo>
-    <!-- <plugin name="gazebo_ros_control" filename="libmy_gazebo_ros_control.so"> -->
-      <plugin name="gazebo_ros_control" filename="libgazebo_ros_control.so">
-      <robotNamespace>/panda</robotNamespace>
-      <!-- <robotSimType>gazebo_ros_control/DefaultRobotHWSim</robotSimType> -->
-    </plugin>
-  </gazebo>
 </robot>
