Commit message: plan execution in hardware

File: ros_ws/src/projects/dexterous_in_hand_manip/manipulation_env/desc/long_block.urdf (robot description, URDF)
Before this commit: robot block_object, 1 links, 0 joints
Links:
- link block: geometry collision box size=0.04 0.025 0.1; visual box size=0.04 0.025 0.1
