Commit message: simulation updates

File: ros_ws/src/projects/dexterous_in_hand_manip/manipulation_env/desc/rectangular_prism.urdf (robot description, URDF)
Before this commit: robot block_object, 1 links, 0 joints
Links:
- link block: geometry collision box size=0.03 0.03 0.08; visual box size=0.03 0.03 0.08

File: ros_ws/src/projects/dexterous_in_hand_manip/manipulation_env/desc/table_box.urdf (robot description, URDF)
Before this commit: robot table_box, 2 links, 1 joints
Links:
- link table: geometry collision box size=0.3 0.5 0.6; visual box size=0.3 0.5 0.6
Joints:
- joint fixed: origin xyz=0.8 0 0.225 rpy=0 0 0 -> xyz=0.4 -0.5 0.3 rpy=0 0 1.5708
