Commit message: added rrbot and depth sensor env

File: ros_ws/src/projects/soft_manipulation/rrbot_sim/rrbot_description/urdf/rrbot.xacro (robot description, xacro)
@@ -96,5 +96,5 @@
 	<box size="${width} ${width} ${height3}"/>
       </geometry>
-      <material name="orange"/>
+      <material name="black"/>
     </visual>
     <inertial>

Commit message: added skeletonization

File: ros_ws/src/projects/soft_manipulation/rrbot_sim/rrbot_description/urdf/rrbot.xacro (robot description, xacro)
@@ -65,5 +65,5 @@
 	<box size="${width} ${width} ${height2}"/>
       </geometry>
-      <material name="black"/>
+      <material name="red"/>
     </visual>
     <inertial>
@@ -96,5 +96,5 @@
 	<box size="${width} ${width} ${height3}"/>
       </geometry>
-      <material name="black"/>
+      <material name="red"/>
     </visual>
     <inertial>

Commit message: Fixed conversions for skeletonization

File: ros_ws/src/projects/soft_manipulation/rrbot_sim/rrbot_description/urdf/rrbot.xacro (robot description, xacro)
@@ -91,4 +91,5 @@
       </geometry>
     </collision>
+<!--
     <visual>
       <origin xyz="0 0 ${height3/2 - axel_offset}" rpy="0 0 0"/>
@@ -97,5 +98,5 @@
       </geometry>
       <material name="red"/>
-    </visual>
+    </visual> -->
     <inertial>
       <origin xyz="0 0 ${height3/2 - axel_offset}" rpy="0 0 0"/>
